File: Theremin-Kicad/Theremin.kicad_pcb (KiCad board)
At the start: 2 copper layers, 131.8 x 80 mm, 36 parts, among them CON1 BARREL_JACK, P1 SENSOR_1_NOTA, P2 SENSOR_2_VOL, P3 FPGA_OUTS, P4 FPGA_INS, P5 AUDIO_OUT, P6 CONN_2, SW1 VOL_UP, SW2 VOL_DOWN, SW3 PITCH_UP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

Commit message: PCB Corregida
Parts:
- SW1, SW2, SW3, SW4, SW5, SW6: footprint SW_PUSH_SMALL_ok -> SW_PUSH_SMALL_NW
- moved R10 0.71 mm to (83.1, 91.5)
- moved R8 0.71 mm to (104.9, 91.4)
Routing:
- net GND: track 448.3 -> 444.2 mm
- net 3.3v: track 67.1 -> 70.6 mm
- net N-0000039: track 10.1 -> 12.1 mm
- net N-0000019: track 7.40 -> 9.24 mm
- net N-0000017: track 7.40 -> 9.23 mm
- net N-0000018: track 7.40 -> 9.23 mm
- net N-0000022: track 7.40 -> 9.18 mm
- net N-0000021: track 3.95 -> 4.54 mm
- net N-0000020: track 4.46 -> 5.05 mm
- net N-0000015: track 4.46 -> 5.05 mm
- net N-0000030: track 50.7 -> 50.1 mm
- net N-0000027: track 32.1 -> 32.7 mm
- net N-000001: track 51.6 -> 51.1 mm
Other:
- net class 6: via_dia 0.889 -> 1.5; via_drill 0.635 -> 0.6
- net class 7: via_dia 0.889 -> 1.5; via_drill 0.635 -> 0.6
- net class 8: via_dia 0.889 -> 1.5; via_drill 0.635 -> 0.6
- net class 9: via_dia 0.889 -> 1.5; via_drill 0.635 -> 0.6
- net class NW added: clearance 0.254, trace_width 0.9, via_dia 1.5, via_drill 0.6
